Commit message: Completati: 1,2,4. 2 serve debug

File: arm_description/urdf/arm.urdf.xacro (robot description, xacro)
@@ -30,5 +30,4 @@
     <child link="base_turn"/>
     <origin xyz="-0.0011 -0.011 0.05"/>
-    <xacro:hardware_interface_for_joint hardware_interface_type="PositionJointInterface"/>
   </joint>
   <link name="base_turn">
@@ -58,5 +57,4 @@
     <axis xyz="0 0 1" />
     <limit effort="300" velocity="0.1" lower="-2.57" upper="2.57"/>
-    <xacro:hardware_interface_for_joint hardware_interface_type="PositionJointInterface"/>
   </joint>
   <link name="base_turn_rot">
@@ -83,5 +81,4 @@
     <child link="dyn2"/>
     <origin xyz="0 0 0.0385" rpy="0 1.57 1.57 "/>
-    <xacro:hardware_interface_for_joint hardware_interface_type="PositionJointInterface"/>
   </joint>
   <link name="dyn2">
@@ -110,5 +107,4 @@
     <axis xyz="0 0 1" />
     <limit effort="300" velocity="0.1" lower="-3.14" upper="3.14"/>
-    <xacro:hardware_interface_for_joint hardware_interface_type="PositionJointInterface"/>
   </joint>
   <link name="dyn2_r">
@@ -118,5 +114,4 @@
     <child link="f4"/>
     <origin xyz="-0.047 0.0 -0.003" rpy="0 1.57 1.57"/>
-    <xacro:hardware_interface_for_joint hardware_interface_type="PositionJointInterface"/>
   </joint>
   <link name="f4">
@@ -144,5 +139,4 @@
     <child link="dyn3"/>
     <origin xyz="-0.004 0.0645 0 " rpy="-1.57 3.14 1.57"/>
-    <xacro:hardware_interface_for_joint hardware_interface_type="PositionJointInterface"/>
   </joint>
   <link name="dyn3">
@@ -171,5 +165,4 @@
     <axis xyz="0 0 1" />
     <limit effort="300" velocity="0.1" lower="-3.14" upper="3.14"/>
-    <xacro:hardware_interface_for_joint hardware_interface_type="PositionJointInterface"/>
   </joint>
  <link name="dyn3_r">
@@ -179,5 +172,4 @@
     <child link="f5"/>
     <origin xyz="-0.046 -0.0 -0.002" rpy="1.57 1.57 3.1415 "/>
-    <xacro:hardware_interface_for_joint hardware_interface_type="PositionJointInterface"/>
   </joint>
   <link name="f5">
@@ -204,5 +196,4 @@
     <child link="dyn4"/>
     <origin xyz="-0.004 0.065 -0.0" rpy="-1.57 3.1415 1.57 "/>
-    <xacro:hardware_interface_for_joint hardware_interface_type="PositionJointInterface"/>
   </joint>
   <link name="dyn4">
@@ -231,5 +222,4 @@
     <axis xyz="0 0 1" />
     <limit effort="300" velocity="0.1" lower="-3.14" upper="3.14"/>
-    <xacro:hardware_interface_for_joint hardware_interface_type="PositionJointInterface"/>
   </joint>
   <link name="dyn4_r">
@@ -239,5 +229,4 @@
     <child link="wrist"/>
     <origin xyz="-0.017 -0.013 0.003" rpy="1.57 1.57 -1.57"/>
-    <xacro:hardware_interface_for_joint hardware_interface_type="PositionJointInterface"/>
   </joint>
   <link name="wrist">
@@ -265,5 +254,4 @@
     <child link="dyn5"/>
     <origin xyz="0.0038 -0.013 0.0275" rpy="0 0 1.57"/>
-    <xacro:hardware_interface_for_joint hardware_interface_type="PositionJointInterface"/>
   </joint>
     <link name="dyn5">
@@ -292,5 +280,4 @@
     <axis xyz="0 0 1" />
     <limit effort="300" velocity="0.1" lower="-3.14" upper="3.14"/>
-    <xacro:hardware_interface_for_joint hardware_interface_type="PositionJointInterface"/>
   </joint>
   <link name="dyn5_r">
@@ -300,5 +287,4 @@
     <child link="crawer_base"/>
     <origin xyz="0.015 0 0.019" rpy="0 0 1.57"/>
-    <xacro:hardware_interface_for_joint hardware_interface_type="PositionJointInterface"/>
   </joint>
   <link name="crawer_base">
@@ -326,5 +312,4 @@
     <child link="crawer_left"/>
     <origin xyz="-0.03 0.015 0.01" rpy="0 -1.57 0"/>
-    <xacro:hardware_interface_for_joint hardware_interface_type="PositionJointInterface"/>
   </joint>
   <link name="crawer_left">
@@ -354,5 +339,4 @@
     <child link="crawer_right"/>
     <origin xyz="0.03 0.015 0.01" rpy="3.1415 -1.57 0"/>
-    <xacro:hardware_interface_for_joint hardware_interface_type="PositionJointInterface"/>
   </joint>
   <link name="crawer_right">
@@ -378,3 +362,26 @@
     </inertial>
   </link>
+  <ros2_control name="IgnitionSystem" type="system">
+    <hardware>
+      <plugin>ign_ros2_control/IgnitionSystem</plugin>
+    </hardware>
+    <joint name="j0">
+      <xacro:PositionJointInterface/>
+    </joint>
+    <joint name="j1">
+      <xacro:PositionJointInterface/>
+    </joint>
+    <joint name="j2">
+      <xacro:PositionJointInterface/>
+    </joint>
+    <joint name="j3">
+      <xacro:PositionJointInterface/>
+    </joint>
+  </ros2_control>
+  <gazebo>
+    <plugin filename="ign_ros2_control-system" name="ign_ros2_control::IgnitionROS2ControlPlugin">
+      <parameters>$(find arm_gazebo)/config/controllers.yaml</parameters>
+      <controller_manager_prefix_node_name>controller_manager</controller_manager_prefix_node_name>
+    </plugin>
+  </gazebo>
 </robot>

File: arm_description/urdf/arm_hardware_interface.xacro (robot description, xacro)
@@ -3,9 +3,14 @@
 <robot xmlns:xacro="http://www.ros.org/wiki/xacro">
   <!-- Macro for a hardware interface for a joint -->
-  <xacro:macro name="hardware_interface_for_joint" params="hardware_interface_type">
-    <ros2_control>
-      <!-- ros2_control hardware interface configuration -->
-      <hardwareInterface>${hardware_interface_type}</hardwareInterface>
-    </ros2_control>
+  <xacro:macro name="PositionJointInterface">
+    <command_interface name="position">
+    </command_interface>
+    <command_interface name="velocity">
+    </command_interface>
+    <command_interface name="effort">
+    </command_interface>
+    <state_interface name="position"/>
+    <state_interface name="velocity"/>
+    <state_interface name="effort"/>
   </xacro:macro>
 </robot>

Commit message: Total project completed for first time

File: arm_description/urdf/arm.urdf.xacro (robot description, xacro)
@@ -3,7 +3,19 @@
   <!-- Include the hardware interface xacro file -->
   <xacro:include filename="$(find arm_description)/urdf/arm_hardware_interface.xacro"/>
+  <xacro:include filename="$(find arm_gazebo)/urdf/arm_camera.xacro"/>
   <material name="red">
     <color rgba="1 0 0 1"/>
   </material>
+  <material name="green">
+    <color rgba="0 1 0 1"/>
+  </material>
+  <material name="blue_debug">
+    <color rgba="0 0 1 0.5"/>
+  </material>
+  <link name="world"/>
+  <joint name="world_to_base_link_joint" type="fixed">
+      <parent link="world"/>
+      <child link="base_link"/>
+  </joint>
   <link name="base_link">
     <visual>
@@ -25,4 +37,19 @@
       <inertia ixx="1.06682889e+08" ixy="0.0" ixz="0.0" iyy="9.92165844e+07" iyz="0.0" izz="1.26939175e+08"/>
     </inertial>
+  </link>
+  <joint name="camera_joint" type="fixed">
+    <parent link="base_link"/>
+    <child link="camera_link"/>
+    <origin xyz="0.0 0.0 0.0" rpy="0.0 0.0 0.0"/>
+  </joint>
+  <link name="camera_link">
+    <visual>
+      <geometry>
+        <!--<box size="0.0000010 0.00000003 0.00000003"/>-->
+        <box size="0.02 0.008 0.008"/>
+      </geometry>
+      <origin rpy="0 0 0" xyz="0 0 -0.022"/>
+      <material name="green"/>
+    </visual>
   </link>
   <joint name="base_1_2" type="fixed">
@@ -366,16 +393,8 @@
       <plugin>ign_ros2_control/IgnitionSystem</plugin>
     </hardware>
-    <joint name="j0">
-      <xacro:PositionJointInterface/>
-    </joint>
-    <joint name="j1">
-      <xacro:PositionJointInterface/>
-    </joint>
-    <joint name="j2">
-      <xacro:PositionJointInterface/>
-    </joint>
-    <joint name="j3">
-      <xacro:PositionJointInterface/>
-    </joint>
+    <xacro:PositionJointInterface name="j0" initial_pos="1.0"/>
+    <xacro:PositionJointInterface name="j1" initial_pos="2.0"/>
+    <xacro:PositionJointInterface name="j2" initial_pos="-1.0"/>
+    <xacro:PositionJointInterface name="j3" initial_pos="-2.0"/>
   </ros2_control>
   <gazebo>
@@ -385,3 +404,23 @@
     </plugin>
   </gazebo>
+  <xacro:arm_camera_plugin/>
+  <gazebo reference="camera_link">
+    <sensor name="camera" type="camera">
+      <camera>
+      <horizontal_fov>1.047</horizontal_fov>
+        <image>
+          <width>320</width>
+          <height>240</height>
+        </image>
+      <clip>
+        <near>0.1</near>
+        <far>100</far>
+      </clip>
+      </camera>
+      <always_on>1</always_on>
+      <update_rate>30</update_rate>
+      <visualize>true</visualize>
+      <topic>camera</topic>
+    </sensor>
+  </gazebo>
 </robot>

File: arm_description/urdf/arm_hardware_interface.xacro (robot description, xacro)
@@ -3,4 +3,5 @@
 <robot xmlns:xacro="http://www.ros.org/wiki/xacro">
   <!-- Macro for a hardware interface for a joint -->
+  <!--
   <xacro:macro name="PositionJointInterface">
     <command_interface name="position">
@@ -10,7 +11,28 @@
     <command_interface name="effort">
     </command_interface>
-    <state_interface name="position"/>
-    <state_interface name="velocity"/>
-    <state_interface name="effort"/>
+    <state_interface name="position">
+      <param name="initial_value">0.0</param>
+    </state_interface>
+    <state_interface name="velocity">
+      <param name="initial_value">0.0</param>
+    </state_interface>
+    <state_interface name="effort">
+      <param name="initial_value">0.0</param>
+    </state_interface>
+  </xacro:macro>
+  -->
+  <xacro:macro name="PositionJointInterface" params="name initial_pos">
+    <joint name="${name}">
+        <command_interface name="position"/>
+        <state_interface name="position">
+            <param name="initial_value">${initial_pos}</param>
+        </state_interface>
+        <state_interface name="velocity">
+            <param name="initial_value">0.0</param>
+        </state_interface>
+        <state_interface name="effort">
+            <param name="initial_value">0.0</param>
+        </state_interface>
+    </joint>
   </xacro:macro>
 </robot>

Commit message: Last version

File: arm_description/urdf/arm.urdf.xacro (robot description, xacro)
@@ -46,5 +46,4 @@
     <visual>
       <geometry>
-        <!--<box size="0.0000010 0.00000003 0.00000003"/>-->
         <box size="0.02 0.008 0.008"/>
       </geometry>
@@ -400,5 +399,5 @@
   <gazebo>
     <plugin filename="ign_ros2_control-system" name="ign_ros2_control::IgnitionROS2ControlPlugin">
-      <parameters>$(find arm_gazebo)/config/controllers.yaml</parameters>
+      <parameters>$(find arm_control)/config/controllers.yaml</parameters>
       <controller_manager_prefix_node_name>controller_manager</controller_manager_prefix_node_name>
     </plugin>

File: arm_description/urdf/arm_hardware_interface.xacro (robot description, xacro)
@@ -1,25 +1,4 @@
 <?xml version="1.0"?>
-<!-- arm_hardware_interface.xacro -->
 <robot xmlns:xacro="http://www.ros.org/wiki/xacro">
-  <!-- Macro for a hardware interface for a joint -->
-  <!--
-  <xacro:macro name="PositionJointInterface">
-    <command_interface name="position">
-    </command_interface>
-    <command_interface name="velocity">
-    </command_interface>
-    <command_interface name="effort">
-    </command_interface>
-    <state_interface name="position">
-      <param name="initial_value">0.0</param>
-    </state_interface>
-    <state_interface name="velocity">
-      <param name="initial_value">0.0</param>
-    </state_interface>
-    <state_interface name="effort">
-      <param name="initial_value">0.0</param>
-    </state_interface>
-  </xacro:macro>
-  -->
   <xacro:macro name="PositionJointInterface" params="name initial_pos">
     <joint name="${name}">
